Commit message: map issue resolved

File: uvd_description/urdf/uvd_new.urdf (robot description, URDF)
Before this commit: robot test_bot, 11 links, 10 joints
Links:
- removed link base
- removed link camera_frame_optical
- removed link uv_base
- removed link uv_top
- added link base_link, mass 100; collision box size=0.4 0.3 0.2; visual box size=0.4 0.3 0.2
- added link realsense_optical_link
- added link robot_footprint
- link imu_link: mass 1e-5 -> 10; geometry collision box size=0.05 0.05 0.05; visual box size=0.05 0.05 0.02
Joints:
- removed joint base_to_back_left_wheel
- removed joint base_to_back_right_wheel
- removed joint base_to_depth_camera
- removed joint base_to_front_left_wheel
- removed joint base_to_front_right_wheel
- removed joint base_to_imu
- removed joint camera_optical_joint
- removed joint uv_base_body
- removed joint uv_base_top
- added joint back_left_wheel_joint: type continuous, parent base_link, child back_left_wheel, origin xyz=-0.175 0.175 0.05 rpy=0 0 0, axis 0 1 0, limit effort=10000 velocity=1000
- added joint back_right_wheel_joint: type continuous, parent base_link, child back_right_wheel, origin xyz=-0.175 -0.175 0.05 rpy=0 0 0, axis 0 1 0, limit effort=10000 velocity=1000
- added joint front_left_wheel_joint: type continuous, parent base_link, child front_left_wheel, origin xyz=0.175 0.175 0.05 rpy=0 0 0, axis 0 1 0, limit effort=10000 velocity=1000
- added joint front_right_wheel_joint: type continuous, parent base_link, child front_right_wheel, origin xyz=0.175 -0.175 0.05 rpy=0 0 0, axis 0 1 0, limit effort=10000 velocity=1000
- added joint imu_joint: type fixed, parent base_link, child imu_link, origin xyz=0 0 0.2 rpy=0 0 0, axis 0 0 0
- added joint realsense_joint: type fixed, parent base_link, child realsense_link, origin xyz=0.14 0 0.675 rpy=0 0 0, axis 0 0 0
- added joint realsense_optical_joint: type fixed, parent realsense_link, child realsense_optical_link, origin xyz=0 0 0 rpy=-1.5707 0 -1.5707
- added joint robot_footprint_joint: type fixed, parent robot_footprint, child base_link, origin xyz=0 0 0 rpy=0 0 0
- joint camera_joint: origin xyz=0.105 0 0 rpy=0 0 0 -> xyz=0.04 0 1.457 rpy=0 0 0; parent uv_top -> base_link

Commit message: Final changes done

File: uvd_description/urdf/uvd_new.urdf (robot description, URDF)
Before this commit: robot robot, 10 links, 9 joints
Links:
- added link uv_base, mass 10; collision cylinder length=1.5 radius=0.095; visual cylinder length=1.5 radius=0.125
Joints:
- added joint uv_base_body: type fixed, parent base_link, child uv_base, origin xyz=0 0 0.85 rpy=0 0 0, axis 0 1 0, limit effort=10000 velocity=1000
- joint camera_joint: origin xyz=0.04 0 1.457 rpy=0 0 0 -> xyz=0.13 0 1.457 rpy=0 0 0
